File: schematic/bluetoothMidiController/bluetoothMidiController.sch (KiCad schematic (older format))
At the start: 26 parts, among them J1 To Feather, J2 Conn_01x06_Female, SW1 OCT-, SW10 G1, SW11 PWR, SW12 G#1, SW13 A1, SW14 A#1, SW15 B1, SW16 C2, SW17 OPT, SW2 OCT+, SW3 C1, SW4 C#1, SW5 D1, SW6 D#1, SW7 E1, SW8 F1, SW9 F#1, U1 MCP23017_SS

Commit message: updated PCB to include two 4.7K resisters for I2C bus
Parts:
- J1: footprint Connector_PinHeader_2.00mm:PinHeader_1x06_P2.00mm_Vertical -> Connector_Wire:SolderWire-0.5sqmm_1x06_P4.8mm_D0.9mm_OD2.3mm
- R2, R3: footprint (none) -> Resistor_SMD:R_1206_3216Metric_Pad1.42x1.75mm_HandSolder
Changed lines of the file:
@@
 EESchema Schematic File Version 4
-LIBS:bluetoothMidiController-cache
-EELAYER 26 0
+EELAYER 30 0
 EELAYER END
 $Descr A4 8268 11693 portrait
@@
 F 0 "J1" V 3900 1150 50  0000 R CNN
 F 1 "To Feather" V 4000 1300 50  0000 R CNN
-F 2 "Connector_PinHeader_2.00mm:PinHeader_1x06_P2.00mm_Vertical" H 3850 1200 50  0001 C CNN
+F 2 "Connector_Wire:SolderWire-0.5sqmm_1x06_P4.8mm_D0.9mm_OD2.3mm" H 3850 1200 50  0001 C CNN
 F 3 "~" H 3850 1200 50  0001 C CNN
 	1    3850 1200
@@
 F 0 "R3" V 5543 2550 50  0000 C CNN
 F 1 "4.7K" V 5634 2550 50  0000 C CNN
-F 2 "" V 5680 2550 50  0001 C CNN
+F 2 "Resistor_SMD:R_1206_3216Metric_Pad1.42x1.75mm_HandSolder" V 5680 2550 50  0001 C CNN
 F 3 "~" H 5750 2550 50  0001 C CNN
 	1    5750 2550
@@
 F 0 "R2" V 5543 2200 50  0000 C CNN
 F 1 "4.7K" V 5634 2200 50  0000 C CNN
-F 2 "" V 5680 2200 50  0001 C CNN
+F 2 "Resistor_SMD:R_1206_3216Metric_Pad1.42x1.75mm_HandSolder" V 5680 2200 50  0001 C CNN
 F 3 "~" H 5750 2200 50  0001 C CNN
 	1    5750 2200
